File: Hardware/PitchDetector.sch (EAGLE design)
At the start: 46 parts, among them IC1 STM32F302CBT6, IC2 LM3940IMP-3.3_NOPB, X1 MINI-USB-32005-201, X2 HD44780LCD-1602, Y1 ABLS-8.000MHZ-K4T

Commit message: Schematic updated.
Connections:
- net 3V3: no longer C19.1, C20.1
- net C3V3: now also C19.1, C20.1
- net CGND: now also C19.2, C20.2
- net GND: no longer C19.2, C20.2
Changed lines of the file:
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@@
-</segment>
-<segment>
-<pinref part="C20" gate="G$1" pin="2"/>
-<pinref part="C19" gate="G$1" pin="2"/>
-<wire x1="137.16" y1="114.3" x2="127" y2="114.3" width="0.1524" layer="91"/>
-<wire x1="127" y1="114.3" x2="127" y2="111.76" width="0.1524" layer="91"/>
-<junction x="127" y="114.3"/>
-<label x="127" y="111.76" size="0.8128" layer="95" rot="R270" xref="yes"/>
 </segment>
 <segment>
@@
 <junction x="38.1" y="121.92"/>
 </segment>
-<segment>
-<pinref part="C19" gate="G$1" pin="1"/>
-<pinref part="C20" gate="G$1" pin="1"/>
-<wire x1="127" y1="121.92" x2="137.16" y2="121.92" width="0.1524" layer="91"/>
-<wire x1="127" y1="121.92" x2="127" y2="124.46" width="0.1524" layer="91"/>
-<junction x="127" y="121.92"/>
-<label x="127" y="124.46" size="0.8128" layer="95" rot="R90" xref="yes"/>
-</segment>
 </net>
 <net name="CGND" class="0">
@@
 <wire x1="60.96" y1="81.28" x2="58.42" y2="81.28" width="0.1524" layer="91"/>
 <label x="58.42" y="81.28" size="0.8128" layer="95" rot="R180" xref="yes"/>
+</segment>
+<segment>
+<pinref part="C20" gate="G$1" pin="2"/>
+<pinref part="C19" gate="G$1" pin="2"/>
+<wire x1="137.16" y1="114.3" x2="127" y2="114.3" width="0.1524" layer="91"/>
+<wire x1="127" y1="114.3" x2="127" y2="111.76" width="0.1524" layer="91"/>
+<junction x="127" y="114.3"/>
+<label x="127" y="111.76" size="0.8128" layer="95" rot="R270" xref="yes"/>
 </segment>
 </net>
@@
 <label x="58.42" y="78.74" size="0.8128" layer="95" rot="R180" xref="yes"/>
 </segment>
-</net>
+<segment>
+<pinref part="C19" gate="G$1" pin="1"/>
+<pinref part="C20" gate="G$1" pin="1"/>
+<wire x1="127" y1="121.92" x2="137.16" y2="121.92" width="0.1524" layer="91"/>
+<wire x1="127" y1="121.92" x2="127" y2="124.46" width="0.1524" layer="91"/>
+<junction x="127" y="121.92"/>
+<label x="127" y="124.46" size="0.8128" layer="95" rot="R90" xref="yes"/>
+</segment>
+</net>

Commit message: Schematic bug fix. PCB updated.
Connections:
- net GND: now also IC1.BOOT0
- net LCD_D4: no longer IC1.PB5
- net LCD_D5: now also IC1.PB5
Changed lines of the file:
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@@
 </variantdefs>
 <classes>
-<class number="0" name="default" width="0" drill="0">
+<class number="0" name="default" width="0.254" drill="0.1">
+<clearance class="0" value="0.1524"/>
 </class>
 </classes>
@@
 <wire x1="71.12" y1="116.84" x2="71.12" y2="119.38" width="0.1524" layer="91"/>
 <label x="71.12" y="119.38" size="0.8128" layer="95" rot="R180" xref="yes"/>
+<pinref part="IC1" gate="G$1" pin="BOOT0"/>
+<wire x1="78.74" y1="116.84" x2="78.74" y2="119.38" width="0.1524" layer="91"/>
+<wire x1="78.74" y1="119.38" x2="71.12" y2="119.38" width="0.1524" layer="91"/>
 </segment>
 <segment>
@@
 <label x="200.66" y="93.98" size="0.8128" layer="95" rot="R270" xref="yes"/>
 </segment>
+<segment>
+<pinref part="IC1" gate="G$1" pin="PB5"/>
+<wire x1="86.36" y1="116.84" x2="86.36" y2="119.38" width="0.1524" layer="91"/>
+<label x="86.36" y="119.38" size="0.8128" layer="95" rot="R90" xref="yes"/>
+</segment>
 </net>
 <net name="LCD_D4" class="0">
@@
 <label x="88.9" y="119.38" size="0.8128" layer="95" rot="R90" xref="yes"/>
 </segment>
-<segment>
-<pinref part="IC1" gate="G$1" pin="PB5"/>
-<wire x1="86.36" y1="116.84" x2="86.36" y2="119.38" width="0.1524" layer="91"/>
-<label x="86.36" y="119.38" size="0.8128" layer="95" rot="R90" xref="yes"/>
-</segment>
-</net>
+</net>

Commit message: Stable board and schematic added.
Connections:
- net 3V3: now also X2.A
- net GND: now also X2.K
Changed lines of the file:
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@@
 </variantdefs>
 <classes>
-<class number="0" name="default" width="0.254" drill="0.1">
+<class number="0" name="default" width="0.254" drill="0.34">
 <clearance class="0" value="0.1524"/>
 </class>
@@
 <wire x1="231.14" y1="96.52" x2="228.6" y2="96.52" width="0.1524" layer="91"/>
 <junction x="228.6" y="96.52"/>
+<pinref part="X2" gate="G$1" pin="K"/>
+<wire x1="190.5" y1="96.52" x2="190.5" y2="109.22" width="0.1524" layer="91"/>
+<wire x1="190.5" y1="109.22" x2="228.6" y2="109.22" width="0.1524" layer="91"/>
+<wire x1="228.6" y1="109.22" x2="228.6" y2="96.52" width="0.1524" layer="91"/>
 </segment>
 <segment>
@@
 <segment>
 <pinref part="X2" gate="G$1" pin="VDD"/>
+<pinref part="X2" gate="G$1" pin="A"/>
+<wire x1="193.04" y1="96.52" x2="193.04" y2="106.68" width="0.1524" layer="91"/>
+<wire x1="193.04" y1="106.68" x2="226.06" y2="106.68" width="0.1524" layer="91"/>
+<wire x1="226.06" y1="106.68" x2="226.06" y2="96.52" width="0.1524" layer="91"/>
 <wire x1="226.06" y1="96.52" x2="226.06" y2="93.98" width="0.1524" layer="91"/>
+<junction x="226.06" y="96.52"/>
 <label x="226.06" y="93.98" size="0.8128" layer="95" rot="R270" xref="yes"/>
 </segment>
@@
 </sheet>
 </sheets>
+<errors>
+</errors>
 </schematic>
 </drawing>
